File: Hardware/Eagle_LEDCUBE.sch (EAGLE design)
At the start: 23 parts

Commit message: main board v2
Parts:
- added C10, C11, C12, C5, C6, C7, C8, C9: (no value), resistor:C-USC0805K
- added IC10, IC11, IC12, IC5, IC6, IC7, IC8, IC9: (no value), TLC5940:IC-PACKAGE_DIL28-1
- added JP12, JP13, JP14, JP15, JP16, JP17, JP18, JP19, JP21, JP22, JP23, JP24, JP25, JP26, JP27, JP28, JP29, JP30, JP32, JP33: (no value), pinhead:PINHD-2X4
- added JP20, JP31: (no value), pinhead:PINHD-2X6
- added R10, R11, R12, R5, R6, R7, R8, R9: 2.2k, resistor:R-US_R0805
Connections:
- removed net SIN_E: IC4.SOUT, JP9.8
- new net 2A1: IC5.OUT0, JP12.1
- new net 2A10: IC5.OUT9, JP13.2
- new net 2A11: IC5.OUT10, JP13.3
- new net 2A12: IC5.OUT11, JP13.4
- new net 2A13: IC5.OUT12, JP13.5
- new net 2A14: IC5.OUT13, JP13.6
- new net 2A15: IC5.OUT14, JP13.7
- new net 2A16: IC5.OUT15, JP13.8
- new net 2A2: IC5.OUT1, JP12.2
- new net 2A3: IC5.OUT2, JP12.3
- new net 2A4: IC5.OUT3, JP12.4
- new net 2A5: IC5.OUT4, JP12.5
- new net 2A6: IC5.OUT5, JP12.6
- new net 2A7: IC5.OUT6, JP12.7
- new net 2A8: IC5.OUT7, JP12.8
- new net 2A9: IC5.OUT8, JP13.1
- new net 2B1: IC6.OUT0, JP14.1
- new net 2B10: IC6.OUT9, JP15.2
- new net 2B11: IC6.OUT10, JP15.3
- new net 2B12: IC6.OUT11, JP15.4
- new net 2B13: IC6.OUT12, JP15.5
- new net 2B14: IC6.OUT13, JP15.6
- new net 2B15: IC6.OUT14, JP15.7
- new net 2B16: IC6.OUT15, JP15.8
- new net 2B2: IC6.OUT1, JP14.2
- new net 2B3: IC6.OUT2, JP14.3
- new net 2B4: IC6.OUT3, JP14.4
- new net 2B5: IC6.OUT4, JP14.5
- new net 2B6: IC6.OUT5, JP14.6
- new net 2B7: IC6.OUT6, JP14.7
- new net 2B8: IC6.OUT7, JP14.8
- new net 2B9: IC6.OUT8, JP15.1
- new net 2C1: IC7.OUT0, JP16.1
- new net 2C10: IC7.OUT9, JP17.2
- new net 2C11: IC7.OUT10, JP17.3
- new net 2C12: IC7.OUT11, JP17.4
- new net 2C13: IC7.OUT12, JP17.5
- new net 2C14: IC7.OUT13, JP17.6
- new net 2C15: IC7.OUT14, JP17.7
- new net 2C16: IC7.OUT15, JP17.8
- new net 2C2: IC7.OUT1, JP16.2
- new net 2C3: IC7.OUT2, JP16.3
- new net 2C4: IC7.OUT3, JP16.4
- new net 2C5: IC7.OUT4, JP16.5
- new net 2C6: IC7.OUT5, JP16.6
- new net 2C7: IC7.OUT6, JP16.7
- new net 2C8: IC7.OUT7, JP16.8
- new net 2C9: IC7.OUT8, JP17.1
- new net 2D1: IC8.OUT0, JP18.1
- new net 2D10: IC8.OUT9, JP19.2
- new net 2D11: IC8.OUT10, JP19.3
- new net 2D12: IC8.OUT11, JP19.4
- new net 2D13: IC8.OUT12, JP19.5
- new net 2D14: IC8.OUT13, JP19.6
- new net 2D15: IC8.OUT14, JP19.7
- new net 2D16: IC8.OUT15, JP19.8
- new net 2D2: IC8.OUT1, JP18.2
- new net 2D3: IC8.OUT2, JP18.3
- new net 2D4: IC8.OUT3, JP18.4
- new net 2D5: IC8.OUT4, JP18.5
- new net 2D6: IC8.OUT5, JP18.6
- new net 2D7: IC8.OUT6, JP18.7
- new net 2D8: IC8.OUT7, JP18.8
- new net 2D9: IC8.OUT8, JP19.1
- new net 2SIN: IC4.SOUT, IC5.SIN, JP20.5, JP9.8
- new net 2SIN_B: IC5.SOUT, IC6.SIN
- new net 2SIN_C: IC6.SOUT, IC7.SIN
- new net 2SIN_D: IC7.SOUT, IC8.SIN
- new net 3A1: IC9.OUT0, JP23.1
- new net 3A10: IC9.OUT9, JP24.2
- new net 3A11: IC9.OUT10, JP24.3
- new net 3A12: IC9.OUT11, JP24.4
- new net 3A13: IC9.OUT12, JP24.5
- new net 3A14: IC9.OUT13, JP24.6
- new net 3A15: IC9.OUT14, JP24.7
- new net 3A16: IC9.OUT15, JP24.8
- new net 3A2: IC9.OUT1, JP23.2
- new net 3A3: IC9.OUT2, JP23.3
- new net 3A4: IC9.OUT3, JP23.4
- new net 3A5: IC9.OUT4, JP23.5
- new net 3A6: IC9.OUT5, JP23.6
- new net 3A7: IC9.OUT6, JP23.7
- new net 3A8: IC9.OUT7, JP23.8
- new net 3A9: IC9.OUT8, JP24.1
- new net 3B1: IC10.OUT0, JP25.1
- new net 3B10: IC10.OUT9, JP26.2
- new net 3B11: IC10.OUT10, JP26.3
- new net 3B12: IC10.OUT11, JP26.4
- new net 3B13: IC10.OUT12, JP26.5
- new net 3B14: IC10.OUT13, JP26.6
- new net 3B15: IC10.OUT14, JP26.7
- new net 3B16: IC10.OUT15, JP26.8
- new net 3B2: IC10.OUT1, JP25.2
- new net 3B3: IC10.OUT2, JP25.3
- new net 3B4: IC10.OUT3, JP25.4
- new net 3B5: IC10.OUT4, JP25.5
- new net 3B6: IC10.OUT5, JP25.6
- new net 3B7: IC10.OUT6, JP25.7
- new net 3B8: IC10.OUT7, JP25.8
- new net 3B9: IC10.OUT8, JP26.1
- new net 3C1: IC11.OUT0, JP27.1
- new net 3C10: IC11.OUT9, JP28.2
- new net 3C11: IC11.OUT10, JP28.3
- new net 3C12: IC11.OUT11, JP28.4
- new net 3C13: IC11.OUT12, JP28.5
- new net 3C14: IC11.OUT13, JP28.6
- new net 3C15: IC11.OUT14, JP28.7
- new net 3C16: IC11.OUT15, JP28.8
- new net 3C2: IC11.OUT1, JP27.2
- new net 3C3: IC11.OUT2, JP27.3
- new net 3C4: IC11.OUT3, JP27.4
- new net 3C5: IC11.OUT4, JP27.5
- new net 3C6: IC11.OUT5, JP27.6
- new net 3C7: IC11.OUT6, JP27.7
- new net 3C8: IC11.OUT7, JP27.8
- new net 3C9: IC11.OUT8, JP28.1
- new net 3D1: IC12.OUT0, JP29.1
- new net 3D10: IC12.OUT9, JP30.2
- new net 3D11: IC12.OUT10, JP30.3
- new net 3D12: IC12.OUT11, JP30.4
- new net 3D13: IC12.OUT12, JP30.5
- new net 3D14: IC12.OUT13, JP30.6
- new net 3D15: IC12.OUT14, JP30.7
- new net 3D16: IC12.OUT15, JP30.8
- new net 3D2: IC12.OUT1, JP29.2
- new net 3D3: IC12.OUT2, JP29.3
- new net 3D4: IC12.OUT3, JP29.4
- new net 3D5: IC12.OUT4, JP29.5
- new net 3D6: IC12.OUT5, JP29.6
- new net 3D7: IC12.OUT6, JP29.7
- new net 3D8: IC12.OUT7, JP29.8
- new net 3D9: IC12.OUT8, JP30.1
- new net 3SIN: IC8.SOUT, IC9.SIN, JP20.8, JP31.5
- new net 3SIN_B: IC10.SIN, IC9.SOUT
- new net 3SIN_C: IC10.SOUT, IC11.SIN
- new net 3SIN_D: IC11.SOUT, IC12.SIN
- new net 4SIN: IC12.SOUT, JP31.8
- new net N$1: IC5.IREF, R5.1
- new net N$2: IC6.IREF, R6.1
- new net N$3: IC7.IREF, R7.1
- new net N$4: IC8.IREF, R8.1
- new net N$6: IC9.IREF, R9.1
- new net N$7: IC10.IREF, R10.1
- new net N$8: IC11.IREF, R11.1
- new net N$9: IC12.IREF, R12.1
- net BLANK: now also IC10.BLANK, IC11.BLANK, IC12.BLANK, IC5.BLANK, IC6.BLANK, IC7.BLANK, IC8.BLANK, IC9.BLANK, JP20.1, JP31.1
- net DCPRG: now also IC10.DCPRG, IC11.DCPRG, IC12.DCPRG, IC5.DCPRG, IC6.DCPRG, IC7.DCPRG, IC8.DCPRG, IC9.DCPRG, JP20.9, JP31.9
- net GND: now also C10.1, C11.1, C12.1, C5.1, C6.1, C7.1, C8.1, C9.1, IC10.GND, IC11.GND, IC12.GND, IC5.GND, IC6.GND, IC7.GND, IC8.GND, IC9.GND, JP20.4, JP31.4, R10.2, R11.2, R12.2, R5.2, R6.2, R7.2, R8.2, R9.2
- net GSCLK: now also IC10.GSCLK, IC11.GSCLK, IC12.GSCLK, IC5.GSCLK, IC6.GSCLK, IC7.GSCLK, IC8.GSCLK, IC9.GSCLK, JP20.2, JP31.2
- net L1: now also JP21.1, JP22.1, JP32.1, JP33.1
- net L2: now also JP21.2, JP22.2, JP32.2, JP33.2
- net L3: now also JP21.3, JP22.3, JP32.3, JP33.3
- net L4: now also JP21.4, JP22.4, JP32.4, JP33.4
- net L5: now also JP21.5, JP22.5, JP32.5, JP33.5
- net L6: now also JP21.6, JP22.6, JP32.6, JP33.6
- net L7: now also JP21.7, JP22.7, JP32.7, JP33.7
- net L8: now also JP21.8, JP22.8, JP32.8, JP33.8
- net SCLK: now also IC10.SCLK, IC11.SCLK, IC12.SCLK, IC5.SCLK, IC6.SCLK, IC7.SCLK, IC8.SCLK, IC9.SCLK, JP20.3, JP31.3
- net VCC: now also C10.2, C11.2, C12.2, C5.2, C6.2, C7.2, C8.2, C9.2, IC10.VCC, IC11.VCC, IC12.VCC, IC5.VCC, IC6.VCC, IC7.VCC, IC8.VCC, IC9.VCC, JP20.6, JP31.6
- net VPRG: now also IC10.VPRG, IC11.VPRG, IC12.VPRG, IC5.VPRG, IC6.VPRG, IC7.VPRG, IC8.VPRG, IC9.VPRG, JP20.10, JP31.10
- net XLAT: now also IC10.XLAT, IC11.XLAT, IC12.XLAT, IC5.XLAT, IC6.XLAT, IC7.XLAT, IC8.XLAT, IC9.XLAT, JP20.7, JP31.7
