File: Hardware/Eagle_LEDCUBE1.brd (EAGLE design)
At the start: 160 x 100 mm, 70 parts

Commit message: adding eagle board 10mm*20mm
Parts:
- removed JP28, JP29, JP30, JP32, JP33, JP7: (no value), pinhead:2X04
- removed JP31: (no value), pinhead:2X06
- added C13: (no value), rcl:C0805K
- added Q1, Q2, Q3, Q4, Q5, Q6, Q7, Q8: SPD30P06P, transistor-fet:TO251AA
- added R13: (no value), rcl:R0805
- added R14, R15, R16, R17, R18, R19, R20, R21: (no value), resistor:R0805
- added S1: (no value), switch-omron:B3F-10XX
- JP1: device pinhead:2X04 -> pinhead:2X06
- JP20, JP9: device pinhead:2X06 -> pinhead:2X04
- moved LPC1 168.7 mm to (21.6, 111.8), turned to 270 degrees
- moved JP6 125.8 mm to (154.9, 2.54)
- moved JP11 93.4 mm to (74.9, 16.5), turned to 90 degrees
- moved JP10 90.6 mm to (52.1, 16.5), flipped to the bottom, turned to 270 degrees
- moved JP22 82.0 mm to (127.0, 53.3), flipped to the bottom, turned to 270 degrees
- moved JP9 81.3 mm to (74.9, 34.3), turned to 90 degrees
- moved JP21 77.0 mm to (149.9, 69.8), turned to 90 degrees
- moved JP20 72.2 mm to (127.0, 68.6), flipped to the bottom, turned to 270 degrees
- moved JP23 67.0 mm to (149.9, 53.3), turned to 90 degrees
- moved JP25 67.0 mm to (149.9, 34.3), turned to 90 degrees
- moved JP27 66.5 mm to (149.9, 16.5), turned to 90 degrees
- moved JP5 61.4 mm to (74.9, 53.3), turned to 90 degrees
- moved JP3 61.1 mm to (74.9, 68.6), turned to 90 degrees
- moved JP24 51.5 mm to (127.0, 34.3), flipped to the bottom, turned to 270 degrees
- moved JP26 50.2 mm to (127.0, 16.5), flipped to the bottom, turned to 270 degrees
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Connections:
- net N$12 renamed VIN
- removed net N$11: LPC1.1
- new net 3.3V: C13.1, LPC1.28, S1.1
- new net LAYER1: LPC1.73, Q1.1
- new net LAYER2: LPC1.72, Q3.1
- new net LAYER3: LPC1.71, Q5.1
- new net LAYER4: LPC1.70, Q7.1
- new net LAYER5: LPC1.69, Q2.1
- new net LAYER6: LPC1.68, Q4.1
- new net LAYER7: LPC1.67, Q6.1
- new net LAYER8: LPC1.66, Q8.1
- new net N$23: Q5.3
- new net N$24: Q7.3
- new net N$25: Q3.3
- new net N$27: Q1.3
- new net N$37: Q8.3
- new net N$38: Q6.3
- new net N$39: Q4.3
- new net N$40: Q2.3
- new net RESET_N: C13.2, LPC1.4, R13.2, S1.4
- net 2SIN: now also JP1.8; no longer JP20.5, JP9.8
- net 3A1: now also JP20.1; no longer JP23.1
- net 3A10: now also JP21.2; no longer JP24.2
- net 3A11: now also JP21.3; no longer JP24.3
- net 3A12: now also JP21.4; no longer JP24.4
- net 3A13: now also JP21.5; no longer JP24.5
- net 3A14: now also JP21.6; no longer JP24.6
- net 3A15: now also JP21.7; no longer JP24.7
- net 3A16: now also JP21.8; no longer JP24.8
- net 3A2: now also JP20.2; no longer JP23.2
- net 3A3: now also JP20.3; no longer JP23.3
- net 3A4: now also JP20.4; no longer JP23.4
- net 3A5: now also JP20.5; no longer JP23.5
- net 3A6: now also JP20.6; no longer JP23.6
- net 3A7: now also JP20.7; no longer JP23.7
- net 3A8: now also JP20.8; no longer JP23.8
- net 3A9: now also JP21.1; no longer JP24.1
- net 3B1: now also JP22.1; no longer JP25.1
- net 3B10: now also JP23.2; no longer JP26.2
- net 3B11: now also JP23.3; no longer JP26.3
- net 3B12: now also JP23.4; no longer JP26.4
- net 3B13: now also JP23.5; no longer JP26.5
- net 3B14: now also JP23.6; no longer JP26.6
- net 3B15: now also JP23.7; no longer JP26.7
- net 3B16: now also JP23.8; no longer JP26.8
- net 3B2: now also JP22.2; no longer JP25.2
- net 3B3: now also JP22.3; no longer JP25.3
- net 3B4: now also JP22.4; no longer JP25.4
- net 3B5: now also JP22.5; no longer JP25.5
- net 3B6: now also JP22.6; no longer JP25.6
- net 3B7: now also JP22.7; no longer JP25.7
- net 3B8: now also JP22.8; no longer JP25.8
- net 3B9: now also JP23.1; no longer JP26.1
- net 3C1: now also JP24.1; no longer JP27.1
- net 3C10: now also JP25.2; no longer JP28.2
- net 3C11: now also JP25.3; no longer JP28.3
- net 3C12: now also JP25.4; no longer JP28.4
- net 3C13: now also JP25.5; no longer JP28.5
- net 3C14: now also JP25.6; no longer JP28.6
- net 3C15: now also JP25.7; no longer JP28.7
- net 3C16: now also JP25.8; no longer JP28.8
- net 3C2: now also JP24.2; no longer JP27.2
- net 3C3: now also JP24.3; no longer JP27.3
- net 3C4: now also JP24.4; no longer JP27.4
- net 3C5: now also JP24.5; no longer JP27.5
- net 3C6: now also JP24.6; no longer JP27.6
- net 3C7: now also JP24.7; no longer JP27.7
- net 3C8: now also JP24.8; no longer JP27.8
- net 3C9: now also JP25.1; no longer JP28.1
- net 3D1: now also JP26.1; no longer JP29.1
- net 3D10: now also JP27.2; no longer JP30.2
- net 3D11: now also JP27.3; no longer JP30.3
- net 3D12: now also JP27.4; no longer JP30.4
- net 3D13: now also JP27.5; no longer JP30.5
- net 3D14: now also JP27.6; no longer JP30.6
- net 3D15: now also JP27.7; no longer JP30.7
- net 3D16: now also JP27.8; no longer JP30.8
- net 3D2: now also JP26.2; no longer JP29.2
- net 3D3: now also JP26.3; no longer JP29.3
- net 3D4: now also JP26.4; no longer JP29.4
- net 3D5: now also JP26.5; no longer JP29.5
- net 3D6: now also JP26.6; no longer JP29.6
- net 3D7: now also JP26.7; no longer JP29.7
- net 3D8: now also JP26.8; no longer JP29.8
- net 3D9: now also JP27.1; no longer JP30.1
- net 3SIN: no longer JP20.8, JP31.5
- net 4SIN: no longer JP31.8
- net A1: now also JP2.1; no longer JP1.1
- net A10: now also JP3.2; no longer JP2.2
- net A11: now also JP3.3; no longer JP2.3
- net A12: now also JP3.4; no longer JP2.4
- net A13: now also JP3.5; no longer JP2.5
- net A14: now also JP3.6; no longer JP2.6
- net A15: now also JP3.7; no longer JP2.7
- net A16: now also JP3.8; no longer JP2.8
- net A2: now also JP2.2; no longer JP1.2
- net A3: now also JP2.3; no longer JP1.3
- net A4: now also JP2.4; no longer JP1.4
- net A5: now also JP2.5; no longer JP1.5
- net A6: now also JP2.6; no longer JP1.6
- net A7: now also JP2.7; no longer JP1.7
- net A8: now also JP2.8; no longer JP1.8
- net A9: now also JP3.1; no longer JP2.1
- net B1: now also JP4.1; no longer JP3.1
- net B10: now also JP5.2; no longer JP4.2
- net B11: now also JP5.3; no longer JP4.3
- net B12: now also JP5.4; no longer JP4.4
- net B13: now also JP5.5; no longer JP4.5
- net B14: now also JP5.6; no longer JP4.6
- net B15: now also JP5.7; no longer JP4.7
- net B16: now also JP5.8; no longer JP4.8
- net B2: now also JP4.2; no longer JP3.2
- net B3: now also JP4.3; no longer JP3.3
- net B4: now also JP4.4; no longer JP3.4
- net B5: now also JP4.5; no longer JP3.5
- net B6: now also JP4.6; no longer JP3.6
- net B7: now also JP4.7; no longer JP3.7
- net B8: now also JP4.8; no longer JP3.8
- net B9: now also JP5.1; no longer JP4.1
- net BLANK: now also JP1.1, LPC1.24; no longer JP20.1, JP31.1, JP9.1
- net C1: now also JP8.1; no longer JP5.1
- net C10: now also JP9.2; no longer JP6.2
- net C11: now also JP9.3; no longer JP6.3
- net C12: now also JP9.4; no longer JP6.4
- net C13: now also JP9.5; no longer JP6.5
- net C14: now also JP9.6; no longer JP6.6
- net C15: now also JP9.7; no longer JP6.7
- net C16: now also JP9.8; no longer JP6.8
- net C2: now also JP8.2; no longer JP5.2
- net C3: now also JP8.3; no longer JP5.3
- net C4: now also JP8.4; no longer JP5.4
- net C5: now also JP8.5; no longer JP5.5
- net C6: now also JP8.6; no longer JP5.6
- net C7: now also JP8.7; no longer JP5.7
- net C8: now also JP8.8; no longer JP5.8
- net C9: now also JP9.1; no longer JP6.1
- net D1: now also JP10.1; no longer JP7.1
- net D10: now also JP11.2; no longer JP8.2
- net D11: now also JP11.3; no longer JP8.3
- net D12: now also JP11.4; no longer JP8.4
- net D13: now also JP11.5; no longer JP8.5
- net D14: now also JP11.6; no longer JP8.6
- net D15: now also JP11.7; no longer JP8.7
- net D16: now also JP11.8; no longer JP8.8
- net D2: now also JP10.2; no longer JP7.2
- net D3: now also JP10.3; no longer JP7.3
- net D4: now also JP10.4; no longer JP7.4
- net D5: now also JP10.5; no longer JP7.5
- net D6: now also JP10.6; no longer JP7.6
- net D7: now also JP10.7; no longer JP7.7
- net D8: now also JP10.8; no longer JP7.8
- net D9: now also JP11.1; no longer JP8.1
- net DCPRG: now also JP1.9, LPC1.26; no longer JP20.9, JP31.9, JP9.9
- net GND: now also JP1.4, LPC1.1, R13.1, R14.1, R15.1, R16.1, R17.1, R18.1, R19.1, R20.1, R21.1; no longer JP20.4, JP31.4, JP9.4
- net GSCLK: now also JP1.2, LPC1.42; no longer JP20.2, JP31.2, JP9.2
- net L1: now also JP6.1, Q1.2, R14.2; no longer JP10.1, JP11.1, JP21.1, JP22.1, JP32.1, JP33.1
- net L2: now also JP6.2, Q3.2, R16.2; no longer JP10.2, JP11.2, JP21.2, JP22.2, JP32.2, JP33.2
- net L3: now also JP6.3, Q5.2, R18.2; no longer JP10.3, JP11.3, JP21.3, JP22.3, JP32.3, JP33.3
- net L4: now also JP6.4, Q7.2, R20.2; no longer JP10.4, JP11.4, JP21.4, JP22.4, JP32.4, JP33.4
- net L5: now also JP6.5, Q2.2, R15.2; no longer JP10.5, JP11.5, JP21.5, JP22.5, JP32.5, JP33.5
- net L6: now also JP6.6, Q4.2, R17.2; no longer JP10.6, JP11.6, JP21.6, JP22.6, JP32.6, JP33.6
- net L7: now also JP6.7, Q6.2, R19.2; no longer JP10.7, JP11.7, JP21.7, JP22.7, JP32.7, JP33.7
- net L8: now also JP6.8, Q8.2, R21.2; no longer JP10.8, JP11.8, JP21.8, JP22.8, JP32.8, JP33.8
- net SCLK: now also JP1.3, LPC1.11; no longer JP20.3, JP31.3, JP9.3
- net SIN: now also JP1.5, LPC1.13; no longer JP9.5
- net VCC: now also JP1.6; no longer JP20.6, JP31.6, JP9.6
- net VPRG: now also JP1.10, LPC1.25; no longer JP20.10, JP31.10, JP9.10
- net XLAT: now also JP1.7, LPC1.23; no longer JP20.7, JP31.7, JP9.7
Routing:
- net N$10: track 666.8 -> 0.00 mm
- net GND: track 0.00 -> 598.1 mm, vias 0 -> 9
- net VPRG: track 0.00 -> 414.4 mm, vias 0 -> 4
- net DCPRG: track 0.00 -> 376.9 mm, vias 0 -> 9
- net XLAT: track 0.00 -> 366.8 mm, vias 0 -> 12
- net GSCLK: track 0.00 -> 349.4 mm, vias 0 -> 14
- net SCLK: track 0.00 -> 345.0 mm, vias 0 -> 9
- net BLANK: track 0.00 -> 339.7 mm, vias 0 -> 12
- net VCC: track 0.00 -> 309.5 mm, vias 0 -> 12
- net L1: track 0.00 -> 144.2 mm
- net L5: track 0.00 -> 128.6 mm, vias 0 -> 2
- net L2: track 0.00 -> 127.4 mm, vias 0 -> 1
- net LAYER8: track 0.00 -> 124.0 mm
- net LAYER4: track 0.00 -> 111.6 mm
- net 2SIN: track 0.00 -> 105.6 mm, vias 0 -> 2
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- added copper zone on layer 1, net GND
- added copper zone on layer 16, net GND
Other:
- board size 160 x 100 mm -> 160 x 97.5 mm
