File: Hardware/Eagle_LEDCUBE1.sch (EAGLE design)
At the start: 69 parts

Commit message: main board v2
Parts:
- added LPC1: (no value), LPCXpresso_boards:LPCXPRESSO_LPC1769
Connections:
- removed net 3SIN_E: IC9.SIN, JP31.5
- new net 4SIN: IC12.SOUT, JP31.8
- new net N$11: LPC1.1
- new net N$12: LPC1.2
- net 3SIN: now also IC9.SIN, JP31.5; no longer IC12.SOUT, JP31.8
Changed lines of the file:
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@@
 <?xml version="1.0" encoding="utf-8"?>
 <!DOCTYPE eagle SYSTEM "eagle.dtd">
-<eagle version="7.1.0">
+<eagle version="6.5.0">
 <drawing>
 <settings>
@@
 <layers>
 <layer number="1" name="Top" color="4" fill="1" visible="no" active="no"/>
+<layer number="2" name="Route2" color="1" fill="3" visible="no" active="no"/>
+<layer number="3" name="Route3" color="4" fill="3" visible="no" active="no"/>
+<layer number="4" name="Route4" color="1" fill="4" visible="no" active="no"/>
+<layer number="5" name="Route5" color="4" fill="4" visible="no" active="no"/>
+<layer number="6" name="Route6" color="1" fill="8" visible="no" active="no"/>
+<layer number="7" name="Route7" color="4" fill="8" visible="no" active="no"/>
+<layer number="8" name="Route8" color="1" fill="2" visible="no" active="no"/>
+<layer number="9" name="Route9" color="4" fill="2" visible="no" active="no"/>
+<layer number="10" name="Route10" color="1" fill="7" visible="no" active="no"/>
+<layer number="11" name="Route11" color="4" fill="7" visible="no" active="no"/>
+<layer number="12" name="Route12" color="1" fill="5" visible="no" active="no"/>
+<layer number="13" name="Route13" color="4" fill="5" visible="no" active="no"/>
+<layer number="14" name="Route14" color="1" fill="6" visible="no" active="no"/>
+<layer number="15" name="Route15" color="4" fill="6" visible="no" active="no"/>
 <layer number="16" name="Bottom" color="1" fill="1" visible="no" active="no"/>
 <layer number="17" name="Pads" color="2" fill="1" visible="no" active="no"/>
@@
 <layer number="48" name="Document" color="7" fill="1" visible="no" active="no"/>
 <layer number="49" name="Reference" color="7" fill="1" visible="no" active="no"/>
+<layer number="50" name="dxf" color="7" fill="1" visible="no" active="no"/>
 <layer number="51" name="tDocu" color="7" fill="1" visible="no" active="no"/>
 <layer number="52" name="bDocu" color="7" fill="1" visible="no" active="no"/>
+<layer number="53" name="tGND_GNDA" color="7" fill="9" visible="no" active="no"/>
+<layer number="54" name="bGND_GNDA" color="1" fill="9" visible="no" active="no"/>
+<layer number="56" name="wert" color="7" fill="1" visible="no" active="no"/>
 <layer number="91" name="Nets" color="2" fill="1" visible="yes" active="yes"/>
 <layer number="92" name="Busses" color="1" fill="1" visible="yes" active="yes"/>
@@
 <layer number="98" name="Guide" color="6" fill="1" visible="yes" active="yes"/>
 <layer number="99" name="SpiceOrder" color="5" fill="1" visible="yes" active="yes"/>
+<layer number="100" name="Muster" color="7" fill="1" visible="yes" active="yes"/>
+<layer number="101" name="Bemassung" color="7" fill="1" visible="yes" active="yes"/>
+<layer number="102" name="bCross" color="7" fill="1" visible="yes" active="yes"/>
+<layer number="103" name="tMap" color="7" fill="1" visible="yes" active="yes"/>
+<layer number="104" name="Name" color="7" fill="1" visible="yes" active="yes"/>
+<layer number="105" name="tPlate" color="7" fill="1" visible="yes" active="yes"/>
+<layer number="106" name="bPlate" color="7" fill="1" visible="yes" active="yes"/>
+<layer number="107" name="Crop" color="7" fill="1" visible="yes" active="yes"/>
+<layer number="116" name="Patch_BOT" color="9" fill="4" visible="yes" active="yes"/>
+<layer number="121" name="_tsilk" color="7" fill="1" visible="yes" active="yes"/>
+<layer number="122" name="_bsilk" color="7" fill="1" visible="yes" active="yes"/>
+<layer number="144" name="Drill_legend" color="7" fill="1" visible="yes" active="yes"/>
+<layer number="151" name="HeatSink" color="7" fill="1" visible="yes" active="yes"/>
+<layer number="199" name="L$199" color="7" fill="1" visible="yes" active="yes"/>
+<layer number="200" name="200bmp" color="7" fill="1" visible="yes" active="yes"/>
+<layer number="201" name="201bmp" color="2" fill="0" visible="yes" active="yes"/>
+<layer number="202" name="202bmp" color="15" fill="1" visible="yes" active="yes"/>
+<layer number="203" name="203bmp" color="0" fill="1" visible="yes" active="yes"/>
+<layer number="204" name="204bmp" color="0" fill="1" visible="yes" active="yes"/>
+<layer number="205" name="205bmp" color="6" fill="10" visible="yes" active="yes"/>
+<layer number="206" name="206bmp" color="7" fill="10" visible="yes" active="yes"/>
+<layer number="207" name="207bmp" color="8" fill="10" visible="yes" active="yes"/>
+<layer number="208" name="208bmp" color="9" fill="10" visible="yes" active="yes"/>
+<layer number="209" name="209bmp" color="7" fill="1" visible="yes" active="yes"/>
+<layer number="210" name="210bmp" color="7" fill="1" visible="yes" active="yes"/>
+<layer number="211" name="211bmp" color="7" fill="1" visible="yes" active="yes"/>
+<layer number="212" name="212bmp" color="7" fill="1" visible="yes" active="yes"/>
+<layer number="213" name="213bmp" color="7" fill="1" visible="yes" active="yes"/>
+<layer number="214" name="214bmp" color="7" fill="1" visible="yes" active="yes"/>
+<layer number="215" name="215bmp" color="7" fill="1" visible="yes" active="yes"/>
+<layer number="216" name="216bmp" color="7" fill="1" visible="yes" active="yes"/>
+<layer number="250" name="Descript" color="3" fill="1" visible="no" active="no"/>
+<layer number="251" name="SMDround" color="12" fill="11" visible="no" active="no"/>
+<layer number="254" name="cooling" color="7" fill="1" visible="yes" active="yes"/>
 </layers>
 <schematic xreflabel="%F%N/%S.%C%R" xrefpart="/%S.%C%R">
@@
 <part name="JP32" library="pinhead" deviceset="PINHD-2X4" device=""/>
 <part name="JP33" library="pinhead" deviceset="PINHD-2X4" device=""/>
+<part name="LPC1" library="LPCXpresso_boards" deviceset="LPCXPRESSO_LPC1769" device=""/>
 </parts>
 <sheets>
@@
 <net name="3SIN" class="0">
 <segment>
-<pinref part="IC8" gate="G$1" pin="SOUT"/>
-<wire x1="215.9" y1="86.36" x2="218.44" y2="86.36" width="0.1524" layer="91"/>
-<label x="220.98" y="86.36" size="1.778" layer="95"/>
-</segment>
-<segment>
 <pinref part="JP20" gate="A" pin="8"/>
 <wire x1="17.78" y1="152.4" x2="25.4" y2="152.4" width="0.1524" layer="91"/>
 <label x="27.94" y="152.4" size="1.778" layer="95"/>
 </segment>
+<segment>
+<pinref part="IC8" gate="G$1" pin="SOUT"/>
+<wire x1="215.9" y1="86.36" x2="218.44" y2="86.36" width="0.1524" layer="91"/>
+<label x="220.98" y="86.36" size="1.778" layer="95"/>
+</segment>
 </net>
 </nets>
@@
 </segment>
 </net>
-<net name="3SIN_E" class="0">
+<net name="3SIN" class="0">
 <segment>
 <pinref part="JP31" gate="A" pin="5"/>
@@
 </segment>
 </net>
-<net name="3SIN" class="0">
+<net name="4SIN" class="0">
 <segment>
 <pinref part="IC12" gate="G$1" pin="SOUT"/>
@@
 </nets>
 </sheet>
+<sheet>
+<description>LPC1769 Board</description>
+<plain>
+</plain>
+<instances>
+<instance part="LPC1" gate="G$1" x="53.34" y="63.5"/>
+</instances>
+<busses>
+</busses>
+<nets>
+<net name="N$11" class="0">
+<segment>
+<pinref part="LPC1" gate="G$1" pin="1"/>
+<wire x1="22.86" y1="99.06" x2="17.78" y2="99.06" width="0.1524" layer="91"/>
+</segment>
+</net>
+<net name="N$12" class="0">
+<segment>
+<pinref part="LPC1" gate="G$1" pin="2"/>
+<wire x1="22.86" y1="96.52" x2="17.78" y2="96.52" width="0.1524" layer="91"/>
+</segment>
+</net>
+</nets>
+</sheet>
 </sheets>
-<errors>
-</errors>
 </schematic>
 </drawing>

Commit message: adding eagle board 10mm*20mm
Parts:
- removed JP28, JP29, JP30, JP32, JP33, JP7: (no value), pinhead:PINHD-2X4
- removed JP31: (no value), pinhead:PINHD-2X6
- added C13: (no value), rcl:C-USC0805K
- added Q1, Q2, Q3, Q4, Q5, Q6, Q7, Q8: SPD30P06P, transistor-fet:SPD30P06P
- added R13: (no value), rcl:R-US_R0805
- added R14, R15, R16, R17, R18, R19, R20, R21: (no value), resistor:R-US_R0805
- added S1: (no value), switch-omron:10-XX
- JP1: device pinhead:PINHD-2X4 -> pinhead:PINHD-2X6
- JP20, JP9: device pinhead:PINHD-2X6 -> pinhead:PINHD-2X4
Connections:
- net N$12 renamed VIN
- removed net N$11: LPC1.1
- new net 3.3V: C13.1, LPC1.28, S1.S
- new net LAYER1: LPC1.73, Q1.G
- new net LAYER2: LPC1.72, Q3.G
- new net LAYER3: LPC1.71, Q5.G
- new net LAYER4: LPC1.70, Q7.G
- new net LAYER5: LPC1.69, Q2.G
- new net LAYER6: LPC1.68, Q4.G
- new net LAYER7: LPC1.67, Q6.G
- new net LAYER8: LPC1.66, Q8.G
- new net N$23: Q5.S
- new net N$24: Q7.S
- new net N$25: Q3.S
- new net N$27: Q1.S
- new net N$37: Q8.S
- new net N$38: Q6.S
- new net N$39: Q4.S
- new net N$40: Q2.S
- new net RESET_N: C13.2, LPC1.4, R13.2, S1.P1
- net 2SIN: now also JP1.8; no longer JP20.5, JP9.8
- net 3A1: now also JP20.1; no longer JP23.1
- net 3A10: now also JP21.2; no longer JP24.2
- net 3A11: now also JP21.3; no longer JP24.3
- net 3A12: now also JP21.4; no longer JP24.4
- net 3A13: now also JP21.5; no longer JP24.5
- net 3A14: now also JP21.6; no longer JP24.6
- net 3A15: now also JP21.7; no longer JP24.7
- net 3A16: now also JP21.8; no longer JP24.8
- net 3A2: now also JP20.2; no longer JP23.2
- net 3A3: now also JP20.3; no longer JP23.3
- net 3A4: now also JP20.4; no longer JP23.4
- net 3A5: now also JP20.5; no longer JP23.5
- net 3A6: now also JP20.6; no longer JP23.6
- net 3A7: now also JP20.7; no longer JP23.7
- net 3A8: now also JP20.8; no longer JP23.8
- net 3A9: now also JP21.1; no longer JP24.1
- net 3B1: now also JP22.1; no longer JP25.1
- net 3B10: now also JP23.2; no longer JP26.2
- net 3B11: now also JP23.3; no longer JP26.3
- net 3B12: now also JP23.4; no longer JP26.4
- net 3B13: now also JP23.5; no longer JP26.5
- net 3B14: now also JP23.6; no longer JP26.6
- net 3B15: now also JP23.7; no longer JP26.7
- net 3B16: now also JP23.8; no longer JP26.8
- net 3B2: now also JP22.2; no longer JP25.2
- net 3B3: now also JP22.3; no longer JP25.3
- net 3B4: now also JP22.4; no longer JP25.4
- net 3B5: now also JP22.5; no longer JP25.5
- net 3B6: now also JP22.6; no longer JP25.6
- net 3B7: now also JP22.7; no longer JP25.7
- net 3B8: now also JP22.8; no longer JP25.8
- net 3B9: now also JP23.1; no longer JP26.1
- net 3C1: now also JP24.1; no longer JP27.1
- net 3C10: now also JP25.2; no longer JP28.2
- net 3C11: now also JP25.3; no longer JP28.3
- net 3C12: now also JP25.4; no longer JP28.4
- net 3C13: now also JP25.5; no longer JP28.5
- net 3C14: now also JP25.6; no longer JP28.6
- net 3C15: now also JP25.7; no longer JP28.7
- net 3C16: now also JP25.8; no longer JP28.8
- net 3C2: now also JP24.2; no longer JP27.2
- net 3C3: now also JP24.3; no longer JP27.3
- net 3C4: now also JP24.4; no longer JP27.4
- net 3C5: now also JP24.5; no longer JP27.5
- net 3C6: now also JP24.6; no longer JP27.6
- net 3C7: now also JP24.7; no longer JP27.7
- net 3C8: now also JP24.8; no longer JP27.8
- net 3C9: now also JP25.1; no longer JP28.1
- net 3D1: now also JP26.1; no longer JP29.1
- net 3D10: now also JP27.2; no longer JP30.2
- net 3D11: now also JP27.3; no longer JP30.3
- net 3D12: now also JP27.4; no longer JP30.4
- net 3D13: now also JP27.5; no longer JP30.5
- net 3D14: now also JP27.6; no longer JP30.6
- net 3D15: now also JP27.7; no longer JP30.7
- net 3D16: now also JP27.8; no longer JP30.8
- net 3D2: now also JP26.2; no longer JP29.2
- net 3D3: now also JP26.3; no longer JP29.3
- net 3D4: now also JP26.4; no longer JP29.4
- net 3D5: now also JP26.5; no longer JP29.5
- net 3D6: now also JP26.6; no longer JP29.6
- net 3D7: now also JP26.7; no longer JP29.7
- net 3D8: now also JP26.8; no longer JP29.8
- net 3D9: now also JP27.1; no longer JP30.1
- net 3SIN: no longer JP20.8, JP31.5
- net 4SIN: no longer JP31.8
- net A1: now also JP2.1; no longer JP1.1
- net A10: now also JP3.2; no longer JP2.2
- net A11: now also JP3.3; no longer JP2.3
- net A12: now also JP3.4; no longer JP2.4
- net A13: now also JP3.5; no longer JP2.5
- net A14: now also JP3.6; no longer JP2.6
- net A15: now also JP3.7; no longer JP2.7
- net A16: now also JP3.8; no longer JP2.8
- net A2: now also JP2.2; no longer JP1.2
- net A3: now also JP2.3; no longer JP1.3
- net A4: now also JP2.4; no longer JP1.4
- net A5: now also JP2.5; no longer JP1.5
- net A6: now also JP2.6; no longer JP1.6
- net A7: now also JP2.7; no longer JP1.7
- net A8: now also JP2.8; no longer JP1.8
- net A9: now also JP3.1; no longer JP2.1
- net B1: now also JP4.1; no longer JP3.1
- net B10: now also JP5.2; no longer JP4.2
- net B11: now also JP5.3; no longer JP4.3
- net B12: now also JP5.4; no longer JP4.4
- net B13: now also JP5.5; no longer JP4.5
- net B14: now also JP5.6; no longer JP4.6
- net B15: now also JP5.7; no longer JP4.7
- net B16: now also JP5.8; no longer JP4.8
- net B2: now also JP4.2; no longer JP3.2
- net B3: now also JP4.3; no longer JP3.3
- net B4: now also JP4.4; no longer JP3.4
- net B5: now also JP4.5; no longer JP3.5
- net B6: now also JP4.6; no longer JP3.6
- net B7: now also JP4.7; no longer JP3.7
- net B8: now also JP4.8; no longer JP3.8
- net B9: now also JP5.1; no longer JP4.1
- net BLANK: now also JP1.1, LPC1.24; no longer JP20.1, JP31.1, JP9.1
- net C1: now also JP8.1; no longer JP5.1
- net C10: now also JP9.2; no longer JP6.2
- net C11: now also JP9.3; no longer JP6.3
- net C12: now also JP9.4; no longer JP6.4
- net C13: now also JP9.5; no longer JP6.5
- net C14: now also JP9.6; no longer JP6.6
- net C15: now also JP9.7; no longer JP6.7
- net C16: now also JP9.8; no longer JP6.8
- net C2: now also JP8.2; no longer JP5.2
- net C3: now also JP8.3; no longer JP5.3
- net C4: now also JP8.4; no longer JP5.4
- net C5: now also JP8.5; no longer JP5.5
- net C6: now also JP8.6; no longer JP5.6
- net C7: now also JP8.7; no longer JP5.7
- net C8: now also JP8.8; no longer JP5.8
- net C9: now also JP9.1; no longer JP6.1
- net D1: now also JP10.1; no longer JP7.1
- net D10: now also JP11.2; no longer JP8.2
- net D11: now also JP11.3; no longer JP8.3
- net D12: now also JP11.4; no longer JP8.4
- net D13: now also JP11.5; no longer JP8.5
- net D14: now also JP11.6; no longer JP8.6
- net D15: now also JP11.7; no longer JP8.7
- net D16: now also JP11.8; no longer JP8.8
- net D2: now also JP10.2; no longer JP7.2
- net D3: now also JP10.3; no longer JP7.3
- net D4: now also JP10.4; no longer JP7.4
- net D5: now also JP10.5; no longer JP7.5
- net D6: now also JP10.6; no longer JP7.6
- net D7: now also JP10.7; no longer JP7.7
- net D8: now also JP10.8; no longer JP7.8
- net D9: now also JP11.1; no longer JP8.1
- net DCPRG: now also JP1.9, LPC1.26; no longer JP20.9, JP31.9, JP9.9
- net GND: now also JP1.4, LPC1.1, R13.1, R14.1, R15.1, R16.1, R17.1, R18.1, R19.1, R20.1, R21.1; no longer JP20.4, JP31.4, JP9.4
- net GSCLK: now also JP1.2, LPC1.42; no longer JP20.2, JP31.2, JP9.2
- net L1: now also JP6.1, Q1.D, R14.2; no longer JP10.1, JP11.1, JP21.1, JP22.1, JP32.1, JP33.1
- net L2: now also JP6.2, Q3.D, R16.2; no longer JP10.2, JP11.2, JP21.2, JP22.2, JP32.2, JP33.2
- net L3: now also JP6.3, Q5.D, R18.2; no longer JP10.3, JP11.3, JP21.3, JP22.3, JP32.3, JP33.3
- net L4: now also JP6.4, Q7.D, R20.2; no longer JP10.4, JP11.4, JP21.4, JP22.4, JP32.4, JP33.4
- net L5: now also JP6.5, Q2.D, R15.2; no longer JP10.5, JP11.5, JP21.5, JP22.5, JP32.5, JP33.5
- net L6: now also JP6.6, Q4.D, R17.2; no longer JP10.6, JP11.6, JP21.6, JP22.6, JP32.6, JP33.6
- net L7: now also JP6.7, Q6.D, R19.2; no longer JP10.7, JP11.7, JP21.7, JP22.7, JP32.7, JP33.7
- net L8: now also JP6.8, Q8.D, R21.2; no longer JP10.8, JP11.8, JP21.8, JP22.8, JP32.8, JP33.8
- net SCLK: now also JP1.3, LPC1.11; no longer JP20.3, JP31.3, JP9.3
- net SIN: now also JP1.5, LPC1.13; no longer JP9.5
- net VCC: now also JP1.6; no longer JP20.6, JP31.6, JP9.6
- net VPRG: now also JP1.10, LPC1.25; no longer JP20.10, JP31.10, JP9.10
- net XLAT: now also JP1.7, LPC1.23; no longer JP20.7, JP31.7, JP9.7
